Commit message: Edits to fix issues regarding erratic behavior - unsuccessful

File: src/crrl_ugv_desc/urdf/crrl_ugv.xacro (robot description, xacro)
@@ -19,4 +19,11 @@
   <xacro:property name="cameraSize" value="0.05"/>
   <xacro:property name="cameraMass" value="0.1"/>
+  <xacro:property name="wheel_kp" value="1.0" />
+  <xacro:property name="wheel_kd" value="1.0" />
+  <xacro:property name="wheel_mu1" value="1" />
+  <xacro:property name="wheel_mu2" value="1" />
+  <xacro:property name="wheel_slip1" value="0.5" />
+  <xacro:property name="wheel_slip2" value="0.1" />
+  <xacro:property name="wheel_gap" value="0.01" />
   <xacro:include filename="$(find crrl_ugv_desc)/urdf/crrl_ugv.gazebo" />
   <xacro:include filename="$(find crrl_ugv_desc)/urdf/materials.xacro" />
@@ -72,9 +79,9 @@
     <child link="elecBox"/>
   </joint>
-  <wheel lr="leftFwd" tY="1" pos="${fWheelPos}"/>
-  <wheel lr="leftCt" tY="1" pos="${cWheelPos}"/>
-  <wheel lr="leftBwd" tY="1" pos="${rWheelPos}"/>
-  <wheel lr="rightFwd" tY="-1" pos="${fWheelPos}"/>
-  <wheel lr="rightCt" tY="-1" pos="${cWheelPos}"/>
-  <wheel lr="rightBwd" tY="-1" pos="${rWheelPos}"/>
+  <wheel lr="leftFwd" tY="1" pos="${fWheelPos}" gap="${wheel_gap}"/>
+  <!-- <wheel lr="leftCt" tY="1" pos="${cWheelPos}"/> -->
+  <wheel lr="leftBwd" tY="1" pos="${rWheelPos}" gap="${wheel_gap}"/>
+  <wheel lr="rightFwd" tY="-1" pos="${fWheelPos}" gap="${wheel_gap*-1}"/>
+  <!-- <wheel lr="rightCt" tY="-1" pos="${cWheelPos}"/> -->
+  <wheel lr="rightBwd" tY="-1" pos="${rWheelPos}" gap="${wheel_gap*-1}"/>
 </robot>

File: src/crrl_ugv_desc/urdf/macros.xacro (robot description, xacro)
@@ -19,5 +19,5 @@
 	      />
   </macro>
-  <macro name="wheel" params="lr tY pos">
+  <macro name="wheel" params="lr tY pos gap">
     <link name="${lr}_wheel">
       <collision>
@@ -27,4 +27,15 @@
 	</geometry>
       </collision>
+      <surface>
+        <friction>
+          <fdir1>1 0 0</fdir1>
+          <kp>${wheel_kp}</kp> <!-- kp and kd for rubber -->
+          <kd>${wheel_kd}</kd>
+          <mu>${wheel_mu1}</mu>
+          <mu2>${wheel_mu2}</mu2>
+          <slip1>${wheel_slip1}</slip1>
+          <slip2>${wheel_slip2}</slip2>
+        </friction>
+      </surface>
       <visual>
 	<origin xyz="0 0 0" rpy="0 ${PI/2} ${PI/2}" />
@@ -41,9 +52,4 @@
     </link>
     <gazebo reference="${lr}_wheel">
-      <mu1 value="1.0"/>
-      <mu2 value="1.0"/>
-      <kp  value="10000000.0" />
-      <kd  value="1.0" />
-      <fdir1 value="1 0 0"/>
       <material>Gazebo/Black</material>
     </gazebo>
@@ -51,8 +57,8 @@
       <parent link="chassis"/>
       <child link="${lr}_wheel"/>
-      <origin xyz="${pos} ${tY*wheelWidth/2+tY*chassisWidth/2} ${wheelRadius}" rpy="0 0 0" />
+      <origin xyz="${pos} ${tY*wheelWidth/2+tY*chassisWidth/2+gap} ${wheelRadius}" rpy="0 0 0" />
       <axis xyz="0 1 0" rpy="0 0 0" />
-      <limit effort="100" velocity="100"/>
-      <joint_properties damping="0.0" friction="0.0"/>
+      <limit effort="0.1" velocity="0.1"/>
+      <joint_properties damping="1.0" friction="1.0"/>
     </joint>
     <transmission name="${lr}_trans">
@@ -63,5 +69,5 @@
       <actuator name="${lr}Motor">
 	<hardwareInterface>EffortJointInterface</hardwareInterface>
-	<mechanicalReduction>10</mechanicalReduction>
+	<mechanicalReduction>1</mechanicalReduction>
       </actuator>
     </transmission>

Commit message: First functional teleoperation. Needs tuning for rotation

File: src/crrl_ugv_desc/urdf/crrl_ugv.xacro (robot description, xacro)
@@ -22,5 +22,5 @@
   <xacro:property name="wheel_kd" value="1.0" />
   <xacro:property name="wheel_mu1" value="1" />
-  <xacro:property name="wheel_mu2" value="1" />
+  <xacro:property name="wheel_mu2" value="0.1" />
   <xacro:property name="wheel_slip1" value="0.5" />
   <xacro:property name="wheel_slip2" value="0.1" />
@@ -80,8 +80,8 @@
   </joint>
   <wheel lr="leftFwd" tY="1" pos="${fWheelPos}" gap="${wheel_gap}"/>
-  <!-- <wheel lr="leftCt" tY="1" pos="${cWheelPos}"/> -->
+  <!-- <wheel lr="leftCt" tY="1" pos="${cWheelPos}" gap="${wheel_gap}"/> -->
   <wheel lr="leftBwd" tY="1" pos="${rWheelPos}" gap="${wheel_gap}"/>
   <wheel lr="rightFwd" tY="-1" pos="${fWheelPos}" gap="${wheel_gap*-1}"/>
-  <!-- <wheel lr="rightCt" tY="-1" pos="${cWheelPos}"/> -->
+  <!-- <wheel lr="rightCt" tY="-1" pos="${cWheelPos}" gap="${wheel_gap*-1}"/> -->
   <wheel lr="rightBwd" tY="-1" pos="${rWheelPos}" gap="${wheel_gap*-1}"/>
 </robot>

File: src/crrl_ugv_desc/urdf/macros.xacro (robot description, xacro)
@@ -59,5 +59,5 @@
       <origin xyz="${pos} ${tY*wheelWidth/2+tY*chassisWidth/2+gap} ${wheelRadius}" rpy="0 0 0" />
       <axis xyz="0 1 0" rpy="0 0 0" />
-      <limit effort="0.1" velocity="0.1"/>
+      <limit effort="100" velocity="100"/>
       <joint_properties damping="1.0" friction="1.0"/>
     </joint>
@@ -69,5 +69,5 @@
       <actuator name="${lr}Motor">
 	<hardwareInterface>EffortJointInterface</hardwareInterface>
-	<mechanicalReduction>1</mechanicalReduction>
+	<mechanicalReduction>10</mechanicalReduction>
       </actuator>
     </transmission>

Commit message: Rotation fix by reducing wheel collision box. 2 Cameras are added to emulate stereo. Temporary fixes

File: src/crrl_ugv_desc/urdf/crrl_ugv.xacro (robot description, xacro)
@@ -17,10 +17,12 @@
   <xacro:property name="cWheelPos" value="0"/>
   <xacro:property name="rWheelPos" value="-0.185"/>
-  <xacro:property name="cameraSize" value="0.05"/>
+  <xacro:property name="cameraSize" value="0.02"/>
   <xacro:property name="cameraMass" value="0.1"/>
+  <xacro:property name="cameraHeight" value="${wheelRadius*2-0.05}"/>
+  <xacro:property name="cameraBaseline" value="0.1"/>
   <xacro:property name="wheel_kp" value="1.0" />
   <xacro:property name="wheel_kd" value="1.0" />
   <xacro:property name="wheel_mu1" value="1" />
-  <xacro:property name="wheel_mu2" value="0.1" />
+  <xacro:property name="wheel_mu2" value="0.5" />
   <xacro:property name="wheel_slip1" value="0.5" />
   <xacro:property name="wheel_slip2" value="0.1" />
@@ -85,3 +87,57 @@
   <!-- <wheel lr="rightCt" tY="-1" pos="${cWheelPos}" gap="${wheel_gap*-1}"/> -->
   <wheel lr="rightBwd" tY="-1" pos="${rWheelPos}" gap="${wheel_gap*-1}"/>
+  <joint name="camera_joint_left" type="fixed">
+    <axis xyz="0 1 0" />
+    <origin xyz="${fWheelPos} ${cameraBaseline*0.5} ${cameraHeight}" rpy="0 0 0"/>
+    <parent link="chassis"/>
+    <child link="camera_link_left"/>
+  </joint>
+  <joint name="camera_joint_right" type="fixed">
+    <axis xyz="0 1 0" />
+    <origin xyz="${fWheelPos} ${-cameraBaseline*0.5} ${cameraHeight}" rpy="0 0 0"/>
+    <parent link="chassis"/>
+    <child link="camera_link_right"/>
+  </joint>
+  <!-- Left Camera -->
+  <link name="camera_link_left">
+    <collision>
+      <origin xyz="0 0 0" rpy="0 0 0"/>
+      <geometry>
+	<box size="${cameraSize} ${cameraSize} ${cameraSize}"/>
+      </geometry>
+    </collision>
+    <visual>
+      <origin xyz="0 0 0" rpy="0 0 0"/>
+      <geometry>
+	<box size="${cameraSize} ${cameraSize} ${cameraSize}"/>
+      </geometry>
+      <material name="red"/>
+    </visual>
+    <inertial>
+      <mass value="1e-5" />
+      <origin xyz="0 0 0" rpy="0 0 0"/>
+      <inertia ixx="1e-6" ixy="0" ixz="0" iyy="1e-6" iyz="0" izz="1e-6" />
+    </inertial>
+  </link>
+    <!-- Left Camera -->
+  <link name="camera_link_right">
+    <collision>
+      <origin xyz="0 0 0" rpy="0 0 0"/>
+      <geometry>
+	<box size="${cameraSize} ${cameraSize} ${cameraSize}"/>
+      </geometry>
+    </collision>
+    <visual>
+      <origin xyz="0 0 0" rpy="0 0 0"/>
+      <geometry>
+	<box size="${cameraSize} ${cameraSize} ${cameraSize}"/>
+      </geometry>
+      <material name="red"/>
+    </visual>
+    <inertial>
+      <mass value="1e-5" />
+      <origin xyz="0 0 0" rpy="0 0 0"/>
+      <inertia ixx="1e-6" ixy="0" ixz="0" iyy="1e-6" iyz="0" izz="1e-6" />
+    </inertial>
+  </link>
 </robot>

File: src/crrl_ugv_desc/urdf/macros.xacro (robot description, xacro)
@@ -19,4 +19,5 @@
 	      />
   </macro>
+  <!-- NOTE: Wheel collision width is reduced to improve turning. Visually accurate -->
   <macro name="wheel" params="lr tY pos gap">
     <link name="${lr}_wheel">
@@ -24,5 +25,5 @@
 	<origin xyz="0 0 0" rpy="0 ${PI/2} ${PI/2}" />
 	<geometry>
-	  <cylinder length="${wheelWidth}" radius="${wheelRadius}"/>
+	  <cylinder length="${wheelWidth*0.01}" radius="${wheelRadius}"/>
 	</geometry>
       </collision>

Commit message: Initial addition of VLP-16 laser scanner

File: src/crrl_ugv_desc/urdf/crrl_ugv.xacro (robot description, xacro)
@@ -28,7 +28,11 @@
   <xacro:property name="wheel_slip2" value="0.1" />
   <xacro:property name="wheel_gap" value="0.01" />
+  <xacro:arg name="gpu" default="false"/>
+  <xacro:property name="gpu" value="$(arg gpu)" />
+  <!-- File includes -->
   <xacro:include filename="$(find crrl_ugv_desc)/urdf/crrl_ugv.gazebo" />
   <xacro:include filename="$(find crrl_ugv_desc)/urdf/materials.xacro" />
   <xacro:include filename="$(find crrl_ugv_desc)/urdf/macros.xacro" />
+  <xacro:include filename="$(find velodyne_description)/urdf/VLP-16.urdf.xacro"/>
   <!-- Robot Definition -->
   <link name="footprint" />
@@ -81,4 +85,9 @@
     <child link="elecBox"/>
   </joint>
+  <!-- VLP-16 to electrical box -->
+  <VLP-16 parent="elecBox" name="velodyne" topic="/velodyne_points" hz="10" samples="440" gpu="${gpu}">
+    <origin xyz="${elecBoxLength/2-chassisLength/2} 0 ${wheelRadius+chassisHeight/2+elecBoxHeight}" rpy="0 0 0" />
+  </VLP-16>
+  <!-- Wheels -->
   <wheel lr="leftFwd" tY="1" pos="${fWheelPos}" gap="${wheel_gap}"/>
   <!-- <wheel lr="leftCt" tY="1" pos="${cWheelPos}" gap="${wheel_gap}"/> -->
@@ -87,4 +96,5 @@
   <!-- <wheel lr="rightCt" tY="-1" pos="${cWheelPos}" gap="${wheel_gap*-1}"/> -->
   <wheel lr="rightBwd" tY="-1" pos="${rWheelPos}" gap="${wheel_gap*-1}"/>
+  <!-- Camera(s) -->
   <joint name="camera_joint_left" type="fixed">
     <axis xyz="0 1 0" />
@@ -120,5 +130,5 @@
     </inertial>
   </link>
-    <!-- Left Camera -->
+  <!-- Right Camera -->
   <link name="camera_link_right">
     <collision>

Commit message: Rviz GUI conf and ZED camera specs added

File: src/crrl_ugv_desc/urdf/crrl_ugv.xacro (robot description, xacro)
@@ -19,6 +19,6 @@
   <xacro:property name="cameraSize" value="0.02"/>
   <xacro:property name="cameraMass" value="0.1"/>
-  <xacro:property name="cameraHeight" value="${wheelRadius*2-0.05}"/>
-  <xacro:property name="cameraBaseline" value="0.1"/>
+  <xacro:property name="cameraHeight" value="${wheelRadius*2-0.025}"/>
+  <xacro:property name="cameraBaseline" value="0.12"/>
   <xacro:property name="wheel_kp" value="1.0" />
   <xacro:property name="wheel_kd" value="1.0" />

Commit message: Warning clean-up

File: src/crrl_ugv_desc/urdf/crrl_ugv.xacro (robot description, xacro)
@@ -3,22 +3,22 @@
   <!-- Properties -->
   <xacro:property name="PI" value="3.1415926535897931"/>
-  <xacro:property name="chassisHeight" value="0.055"/>
-  <xacro:property name="chassisLength" value="0.44"/>
-  <xacro:property name="chassisWidth" value="0.31"/>
-  <xacro:property name="chassisMass" value="10"/>
-  <xacro:property name="elecBoxHeight" value="0.13"/>
-  <xacro:property name="elecBoxLength" value="0.18"/>
-  <xacro:property name="elecBoxWidth" value="0.31"/>
-  <xacro:property name="elecBoxMass" value="2"/>
-  <xacro:property name="wheelWidth" value="0.1"/>
-  <xacro:property name="wheelRadius" value="0.085"/>
-  <xacro:property name="wheelMass" value="0.1"/>
-  <xacro:property name="fWheelPos" value="0.185"/>
-  <xacro:property name="cWheelPos" value="0"/>
-  <xacro:property name="rWheelPos" value="-0.185"/>
-  <xacro:property name="cameraSize" value="0.02"/>
-  <xacro:property name="cameraMass" value="0.1"/>
-  <xacro:property name="cameraHeight" value="${wheelRadius*2-0.025}"/>
-  <xacro:property name="cameraBaseline" value="0.12"/>
+  <xacro:property name="chassis_height" value="0.055"/>
+  <xacro:property name="chassis_length" value="0.44"/>
+  <xacro:property name="chassis_width" value="0.31"/>
+  <xacro:property name="chassis_mass" value="10"/>
+  <xacro:property name="elec_box_height" value="0.13"/>
+  <xacro:property name="elec_box_length" value="0.18"/>
+  <xacro:property name="elec_box_width" value="0.31"/>
+  <xacro:property name="elec_box_mass" value="2"/>
+  <xacro:property name="wheel_width" value="0.1"/>
+  <xacro:property name="wheel_radius" value="0.085"/>
+  <xacro:property name="wheel_mass" value="0.1"/>
+  <xacro:property name="front_wheel_pos" value="0.185"/>
+  <xacro:property name="center_wheel_pos" value="0"/>
+  <xacro:property name="rear_wheel_pos" value="-0.185"/>
+  <xacro:property name="camera_size" value="0.02"/>
+  <xacro:property name="camera_mass" value="0.1"/>
+  <xacro:property name="camera_height" value="${wheel_radius*2-0.025}"/>
+  <xacro:property name="camera_baseline" value="0.12"/>
   <xacro:property name="wheel_kp" value="1.0" />
   <xacro:property name="wheel_kd" value="1.0" />
@@ -43,40 +43,40 @@
   <link name='chassis'>
     <collision>
-      <origin xyz="0 0 ${wheelRadius}" rpy="0 0 0"/>
+      <origin xyz="0 0 ${wheel_radius}" rpy="0 0 0"/>
       <geometry>
-	<box size="${chassisLength} ${chassisWidth} ${chassisHeight}"/>
+	<box size="${chassis_length} ${chassis_width} ${chassis_height}"/>
       </geometry>
     </collision>
     <visual>
-      <origin xyz="0 0 ${wheelRadius}" rpy="0 0 0"/>
+      <origin xyz="0 0 ${wheel_radius}" rpy="0 0 0"/>
       <geometry>
-	<box size="${chassisLength} ${chassisWidth} ${chassisHeight}"/>
+	<box size="${chassis_length} ${chassis_width} ${chassis_height}"/>
       </geometry>
       <material name="orange"/>
     </visual>
     <inertial>
-      <origin xyz="0 0 ${wheelRadius}" rpy="0 0 0"/>
-      <mass value="${chassisMass}"/>
-      <box_inertia m="${chassisMass}" x="${chassisLength}" y="${chassisWidth}" z="${chassisHeight}"/>
+      <origin xyz="0 0 ${wheel_radius}" rpy="0 0 0"/>
+      <mass value="${chassis_mass}"/>
+      <box_inertia m="${chassis_mass}" x="${chassis_length}" y="${chassis_width}" z="${chassis_height}"/>
     </inertial>
   </link>
   <link name='elecBox'>
     <collision>
-      <origin xyz="${elecBoxLength/2-chassisLength/2} 0 ${wheelRadius+chassisHeight/2+elecBoxHeight/2}" rpy="0 0 0"/>
+      <origin xyz="${elec_box_length/2-chassis_length/2} 0 ${wheel_radius+chassis_height/2+elec_box_height/2}" rpy="0 0 0"/>
       <geometry>
-	<box size="${elecBoxLength} ${elecBoxWidth} ${elecBoxHeight}"/>
+	<box size="${elec_box_length} ${elec_box_width} ${elec_box_height}"/>
       </geometry>
     </collision>
     <visual>
-      <origin xyz="${elecBoxLength/2-chassisLength/2} 0 ${wheelRadius+chassisHeight/2+elecBoxHeight/2}" rpy="0 0 0"/>
+      <origin xyz="${elec_box_length/2-chassis_length/2} 0 ${wheel_radius+chassis_height/2+elec_box_height/2}" rpy="0 0 0"/>
        <geometry>
-	<box size="${elecBoxLength} ${elecBoxWidth} ${elecBoxHeight}"/>
+	<box size="${elec_box_length} ${elec_box_width} ${elec_box_height}"/>
       </geometry>
       <material name="orange"/>
     </visual>
     <inertial>
-      <origin xyz="${elecBoxLength/2-chassisLength/2} 0 ${wheelRadius+chassisHeight/2+elecBoxHeight/2}" rpy="0 0 0"/>
-      <mass value="${elecBoxMass}"/>
-      <box_inertia m="${elecBoxMass}" x="${elecBoxLength}" y="${elecBoxWidth}" z="${elecBoxHeight}"/>
+      <origin xyz="${elec_box_length/2-chassis_length/2} 0 ${wheel_radius+chassis_height/2+elec_box_height/2}" rpy="0 0 0"/>
+      <mass value="${elec_box_mass}"/>
+      <box_inertia m="${elec_box_mass}" x="${elec_box_length}" y="${elec_box_width}" z="${elec_box_height}"/>
     </inertial>
   </link>
@@ -87,17 +87,17 @@
   <!-- VLP-16 to electrical box -->
   <VLP-16 parent="elecBox" name="velodyne" topic="/velodyne_points" hz="10" samples="440" gpu="${gpu}">
-    <origin xyz="${elecBoxLength/2-chassisLength/2} 0 ${wheelRadius+chassisHeight/2+elecBoxHeight}" rpy="0 0 0" />
+    <origin xyz="${elec_box_length/2-chassis_length/2} 0 ${wheel_radius+chassis_height/2+elec_box_height}" rpy="0 0 0" />
   </VLP-16>
   <!-- Wheels -->
-  <wheel lr="leftFwd" tY="1" pos="${fWheelPos}" gap="${wheel_gap}"/>
-  <wheel lr="leftCt" tY="1" pos="${cWheelPos}" gap="${wheel_gap}"/>
-  <wheel lr="leftBwd" tY="1" pos="${rWheelPos}" gap="${wheel_gap}"/>
-  <wheel lr="rightFwd" tY="-1" pos="${fWheelPos}" gap="${wheel_gap*-1}"/>
-  <wheel lr="rightCt" tY="-1" pos="${cWheelPos}" gap="${wheel_gap*-1}"/>
-  <wheel lr="rightBwd" tY="-1" pos="${rWheelPos}" gap="${wheel_gap*-1}"/>
+  <wheel lr="leftFwd" tY="1" pos="${front_wheel_pos}" gap="${wheel_gap}"/>
+  <wheel lr="leftCt" tY="1" pos="${center_wheel_pos}" gap="${wheel_gap}"/>
+  <wheel lr="leftBwd" tY="1" pos="${rear_wheel_pos}" gap="${wheel_gap}"/>
+  <wheel lr="rightFwd" tY="-1" pos="${front_wheel_pos}" gap="${wheel_gap*-1}"/>
+  <wheel lr="rightCt" tY="-1" pos="${center_wheel_pos}" gap="${wheel_gap*-1}"/>
+  <wheel lr="rightBwd" tY="-1" pos="${rear_wheel_pos}" gap="${wheel_gap*-1}"/>
   <!-- Camera(s) -->
   <joint name="camera_joint_left" type="fixed">
     <axis xyz="0 1 0" />
-    <origin xyz="${fWheelPos} ${cameraBaseline*0.5} ${cameraHeight}" rpy="0 0 0"/>
+    <origin xyz="${front_wheel_pos} ${camera_baseline*0.5} ${camera_height}" rpy="0 0 0"/>
     <parent link="chassis"/>
     <child link="camera_link_left"/>
@@ -105,5 +105,5 @@
   <joint name="camera_joint_right" type="fixed">
     <axis xyz="0 1 0" />
-    <origin xyz="${fWheelPos} ${-cameraBaseline*0.5} ${cameraHeight}" rpy="0 0 0"/>
+    <origin xyz="${front_wheel_pos} ${-camera_baseline*0.5} ${camera_height}" rpy="0 0 0"/>
     <parent link="chassis"/>
     <child link="camera_link_right"/>
@@ -114,5 +114,5 @@
       <origin xyz="0 0 0" rpy="0 0 0"/>
       <geometry>
-	<box size="${cameraSize} ${cameraSize} ${cameraSize}"/>
+	<box size="${camera_size} ${camera_size} ${camera_size}"/>
       </geometry>
     </collision>
@@ -120,5 +120,5 @@
       <origin xyz="0 0 0" rpy="0 0 0"/>
       <geometry>
-	<box size="${cameraSize} ${cameraSize} ${cameraSize}"/>
+	<box size="${camera_size} ${camera_size} ${camera_size}"/>
       </geometry>
       <material name="red"/>
@@ -135,5 +135,5 @@
       <origin xyz="0 0 0" rpy="0 0 0"/>
       <geometry>
-	<box size="${cameraSize} ${cameraSize} ${cameraSize}"/>
+	<box size="${camera_size} ${camera_size} ${camera_size}"/>
       </geometry>
     </collision>
@@ -141,5 +141,5 @@
       <origin xyz="0 0 0" rpy="0 0 0"/>
       <geometry>
-	<box size="${cameraSize} ${cameraSize} ${cameraSize}"/>
+	<box size="${camera_size} ${camera_size} ${camera_size}"/>
       </geometry>
       <material name="red"/>

File: src/crrl_ugv_desc/urdf/macros.xacro (robot description, xacro)
@@ -1,29 +1,29 @@
 <?xml version="1.0"?>
 <robot name="crrl_ugv" xmlns:xacro="http://www.ros.org/wiki/xacro">
-  <macro name="cylinder_inertia" params="m r h">
+  <xacro:macro name="cylinder_inertia" params="m r h">
     <inertia ixx="${m*(3*r*r+h*h)/12}" ixy = "0" ixz = "0"
 	     iyy="${m*(3*r*r+h*h)/12}" iyz = "0"
              izz="${m*r*r/2}"
 	     />
-  </macro>
-  <macro name="box_inertia" params="m x y z">
+  </xacro:macro>
+  <xacro:macro name="box_inertia" params="m x y z">
     <inertia  ixx="${m*(y*y+z*z)/12}" ixy = "0" ixz = "0"
 	      iyy="${m*(x*x+z*z)/12}" iyz = "0"
 	      izz="${m*(x*x+z*z)/12}"
 	      />
-  </macro>
-  <macro name="sphere_inertia" params="m r">
+  </xacro:macro>
+  <xacro:macro name="sphere_inertia" params="m r">
     <inertia  ixx="${2*m*r*r/5}" ixy = "0" ixz = "0"
 	      iyy="${2*m*r*r/5}" iyz = "0"
 	      izz="${2*m*r*r/5}"
 	      />
-  </macro>
+  </xacro:macro>
   <!-- NOTE: Wheel collision width is reduced to improve turning. Visually accurate -->
-  <macro name="wheel" params="lr tY pos gap">
+  <xacro:macro name="wheel" params="lr tY pos gap">
     <link name="${lr}_wheel">
       <collision>
 	<origin xyz="0 0 0" rpy="0 ${PI/2} ${PI/2}" />
 	<geometry>
-	  <cylinder length="${wheelWidth*0.01}" radius="${wheelRadius}"/>
+	  <cylinder length="${wheel_width*0.01}" radius="${wheel_radius}"/>
 	</geometry>
       </collision>
@@ -42,5 +42,5 @@
 	<origin xyz="0 0 0" rpy="0 ${PI/2} ${PI/2}" />
 	<geometry>
-	  <cylinder length="${wheelWidth}" radius="${wheelRadius}"/>
+	  <cylinder length="${wheel_width}" radius="${wheel_radius}"/>
 	</geometry>
 	<material name="black"/>
@@ -48,6 +48,6 @@
       <inertial>
 	<origin xyz="0 0 0" rpy="0 ${PI/2} ${PI/2}" />
-	<mass value="${wheelMass}"/>
-	<cylinder_inertia m="${wheelMass}" r="${wheelRadius}" h="${wheelWidth}"/>
+	<mass value="${wheel_mass}"/>
+	<cylinder_inertia m="${wheel_mass}" r="${wheel_radius}" h="${wheel_width}"/>
       </inertial>
     </link>
@@ -58,5 +58,5 @@
       <parent link="chassis"/>
       <child link="${lr}_wheel"/>
-      <origin xyz="${pos} ${tY*wheelWidth/2+tY*chassisWidth/2+gap} ${wheelRadius}" rpy="0 0 0" />
+      <origin xyz="${pos} ${tY*wheel_width/2+tY*chassis_width/2+gap} ${wheel_radius}" rpy="0 0 0" />
       <axis xyz="0 1 0" rpy="0 0 0" />
       <limit effort="100" velocity="100"/>
@@ -73,4 +73,4 @@
       </actuator>
     </transmission>
-  </macro>
+  </xacro:macro>
 </robot>

Commit message: Name standardization, world launch file for MTC5 basement

File: src/crrl_ugv_desc/urdf/crrl_ugv.xacro (robot description, xacro)
@@ -36,10 +36,10 @@
   <xacro:include filename="$(find velodyne_description)/urdf/VLP-16.urdf.xacro"/>
   <!-- Robot Definition -->
-  <link name="footprint" />
+  <link name="base_footprint"/>
   <joint name="base_joint" type="fixed">
-    <parent link="footprint"/>
-    <child link="chassis"/>
+    <parent link="base_footprint"/>
+    <child link="base_link"/>
   </joint>
-  <link name='chassis'>
+  <link name='base_link'>
     <collision>
       <origin xyz="0 0 ${wheel_radius}" rpy="0 0 0"/>
@@ -81,6 +81,6 @@
     </inertial>
   </link>
-  <joint name="elec_chassis" type="fixed">
-    <parent link="chassis"/>
+  <joint name="elec_base_link" type="fixed">
+    <parent link="base_link"/>
     <child link="elecBox"/>
   </joint>
@@ -100,5 +100,5 @@
     <axis xyz="0 1 0" />
     <origin xyz="${front_wheel_pos} ${camera_baseline*0.5} ${camera_height}" rpy="0 0 0"/>
-    <parent link="chassis"/>
+    <parent link="base_link"/>
     <child link="camera_link_left"/>
   </joint>
@@ -106,5 +106,5 @@
     <axis xyz="0 1 0" />
     <origin xyz="${front_wheel_pos} ${-camera_baseline*0.5} ${camera_height}" rpy="0 0 0"/>
-    <parent link="chassis"/>
+    <parent link="base_link"/>
     <child link="camera_link_right"/>
   </joint>

File: src/crrl_ugv_desc/urdf/macros.xacro (robot description, xacro)
@@ -56,5 +56,5 @@
     </gazebo>
     <joint name="${lr}_wheel_hinge" type="continuous">
-      <parent link="chassis"/>
+      <parent link="base_link"/>
       <child link="${lr}_wheel"/>
       <origin xyz="${pos} ${tY*wheel_width/2+tY*chassis_width/2+gap} ${wheel_radius}" rpy="0 0 0" />
