Commit message: Added basic IMU

File: src/crrl_ugv_desc/urdf/crrl_ugv.xacro (robot description, xacro)
@@ -28,4 +28,7 @@
   <xacro:property name="wheel_slip2" value="0.1" />
   <xacro:property name="wheel_gap" value="0.01" />
+  <xacro:property name="imu_xoffset" value="0" />
+  <xacro:property name="imu_yoffset" value="0" />
+  <xacro:property name="imu_zoffset" value="0" />
   <xacro:arg name="gpu" default="false"/>
   <xacro:property name="gpu" value="$(arg gpu)" />
@@ -84,4 +87,30 @@
     <parent link="base_link"/>
     <child link="elecBox"/>
+  </joint>
+  <!-- IMU attachment -->
+  <link name="imu_link">
+    <inertial>
+      <mass value="0.001"/>
+      <origin rpy="0 0 0" xyz="0 0 0"/>
+      <inertia ixx="0.0001" ixy="0" ixz="0" iyy="0.000001" iyz="0" izz="0.0001"/>
+    </inertial>
+    <visual>
+      <origin rpy="0 0 0" xyz="0 0 0"/>
+      <geometry>
+	<box size="0.001 0.001 0.001"/>  <!-- <box size="0.001 0.001 0.001"/> -->
+      </geometry>
+    </visual>
+    <collision>
+      <origin rpy="0 0 0" xyz="0 0 0"/>
+      <geometry>
+	<box size=".001 .001 .001"/>
+      </geometry>
+    </collision>
+  </link>
+  <joint name="imu_joint" type="fixed">
+    <axis xyz="1 0 0"/> <!-- 0 1 0 -->
+    <origin xyz="${elec_box_length/2-chassis_length/2+imu_xoffset} ${imu_yoffset} ${wheel_radius+chassis_height/2+elec_box_height/2+imu_zoffset}"/>
+    <parent link="elecBox"/>
+    <child link="imu_link"/>
   </joint>
   <!-- VLP-16 to electrical box -->

Commit message: Stereo enhancements

File: src/crrl_ugv_desc/urdf/crrl_ugv.xacro (robot description, xacro)
@@ -21,4 +21,7 @@
   <xacro:property name="camera_height" value="${wheel_radius*2-0.025}"/>
   <xacro:property name="camera_baseline" value="0.12"/>
+  <xacro:property name="stcam_width" value="${camera_baseline+(camera_size)*2}"/>
+  <xacro:property name="stcam_height" value="${camera_size*2}"/>
+  <xacro:property name="stcam_depth" value="${camera_size*2}"/>
   <xacro:property name="wheel_kp" value="1.0" />
   <xacro:property name="wheel_kd" value="1.0" />
@@ -126,14 +129,35 @@
   <wheel lr="rightBwd" tY="-1" pos="${rear_wheel_pos}" gap="${wheel_gap*-1}"/>
   <!-- Camera(s) -->
+  <joint name="camera_joint" type="fixed">
+    <axis xyz="0 1 0" />
+    <origin xyz="${front_wheel_pos} 0 ${camera_height}" rpy="0 0 0"/>
+    <parent link="base_link"/>
+    <child link="camera_link"/>
+  </joint>
+  <link name="camera_link">
+    <collision>
+      <origin xyz="0 0 0" rpy="0 0 0"/>
+      <geometry>
+	<box size="${stcam_height} ${stcam_width} ${stcam_depth}"/>
+      </geometry>
+    </collision>
+    <visual>
+      <origin xyz="0 0 0" rpy="0 0 0"/>
+      <geometry>
+	<box size="${stcam_height} ${stcam_width} ${stcam_depth}"/>
+      </geometry>
+      <material name="blue"/>
+    </visual>
+  </link>
   <joint name="camera_joint_left" type="fixed">
     <axis xyz="0 1 0" />
-    <origin xyz="${front_wheel_pos} ${camera_baseline*0.5} ${camera_height}" rpy="0 0 0"/>
-    <parent link="base_link"/>
+    <origin xyz="${stcam_depth/2} ${camera_baseline*0.5} 0" rpy="0 0 0"/>
+    <parent link="camera_link"/>
     <child link="camera_link_left"/>
   </joint>
   <joint name="camera_joint_right" type="fixed">
     <axis xyz="0 1 0" />
-    <origin xyz="${front_wheel_pos} ${-camera_baseline*0.5} ${camera_height}" rpy="0 0 0"/>
-    <parent link="base_link"/>
+    <origin xyz="${stcam_depth/2} ${-camera_baseline*0.5} 0" rpy="0 0 0"/>
+    <parent link="camera_link"/>
     <child link="camera_link_right"/>
   </joint>
